File: hardware/STEP800_r1_0_0.brd (EAGLE design)
At the start: 120 x 100 mm, 276 parts, among them IC1 0982_W5500LONG, J1 POWERJACK, J10 691321300004, J11 691321300004, J12 691321300004, J3 CONN_06_SMD_FEMALE, J4 SDCARD_SLOT_TF-115K, J5 691321300004, J6 691321300004, J7 691321300004, J8 691321300004, J9 691321300004, Q1 FDD4141TO252, Q2 32.768kHz, U1 74HC165PW, U2 USBLC6-2SC6, U3 74HC595, U4 LD1117S33, U5 ATSAMD21G-A, X1 CONN_02, X2 25MHz, X3 RJ45_MAGNETICS_LED_HR871181A

Commit message: Updated hardware design files
Parts:
- added R22: 330R, OPL_Resistor:R0603
- added TP40, TP41, TP42: TESTPOINT_D1.6, PonoorExperiments:TESTPOINT_D1.6
- C105, C107, C109, C111, C65, C67, C69, C71: value 220nF -> 220nf; device Seeed-Capacitor:C0402 -> OPL_Capacitor:C0603
- C23, C28: device Seeed-Capacitor:C0402 -> OPL_Capacitor:C0603
- R3, R5, R9: value 10K 1/10W -> 100K 1/10W
- TP7: value TESTPOINT_3X1 -> TESTPOINT_D1.6; device PonoorExperiments:TESTPOINT_3X1 -> PonoorExperiments:TESTPOINT_D1.6
- moved TP7 100.0 mm to (111.8, 66.0), turned to 0 degrees
- moved RN4 5.21 mm to (26.0, 72.0)
- moved R13 5.08 mm to (16.5, 86.4), turned to 90 degrees
- moved R12 4.02 mm to (16.5, 83.8)
- moved C28 3.99 mm to (21.8, 75.7), turned to 180 degrees
- moved C30 3.92 mm to (21.8, 73.0), turned to 270 degrees
- moved C27 3.81 mm to (21.3, 70.4), turned to 180 degrees
- moved C29 3.63 mm to (21.3, 78.4), turned to 270 degrees
- moved TP6 2.54 mm to (16.5, 35.6)
- moved RN5 2.44 mm to (21.8, 81.3)
- moved X3 1.78 mm to (8.89, 73.7)
- moved R11 0.76 mm to (21.7, 67.3)
- moved L1 0.64 mm to (24.0, 67.3)
- moved R9 0.51 mm to (26.3, 54.1)
- moved C18 0.25 mm to (26.9, 67.3)
Connections:
- removed net D2: TP7.P$1, U5.23
- new net 74HC165_MOSI: U1.10, U5.23
- new net N$46: 3.3V.+, R22.1
- net GND: no longer U1.10
- net N$27: now also R22.2; no longer 3.3V.+
- net N$34: now also TP7.1
- net N$40: now also TP40.1
- net N$42: now also TP41.1
- net N$44: now also TP42.1
Routing:
- net D2: track 19.5 -> 0.00 mm, vias 1 -> 0
- net 74HC165_MOSI: track 0.00 -> 13.4 mm, vias 0 -> 3
- net TX_P: track 21.2 -> 14.0 mm
- net TX_N: track 21.8 -> 15.0 mm
- net TXO_N: track 14.1 -> 20.3 mm
- net N$9: track 19.2 -> 13.3 mm
- net +3V3A: track 69.0 -> 74.8 mm
- net RXI_N: track 6.29 -> 11.9 mm
- net RX_N: track 17.1 -> 11.8 mm
- net RX_P: track 15.5 -> 10.3 mm
- net 3.3V: track 416.3 -> 421.4 mm
- net N$8: track 26.1 -> 21.0 mm
- net N$7: track 10.6 -> 15.2 mm
- net TXO_P: track 13.6 -> 18.1 mm
- net N$46: track 0.00 -> 4.18 mm
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Other:
- board text added: "2021-04-28"
- board text added: "STEP800 r1.0.0"
- board text added: "rev.1.0.0"
- board text removed: "D2"
- board text removed: "STEP800 proto r0.4.0"
- board text removed: "rev.0.4.0"
- board text removed: "rev.2021-04-13"
