File: hardware/STEP800_r1_0_0.sch (EAGLE design)
At the start: 271 parts, among them IC1 0982_W5500LONG, J1 POWERJACK, J10 691321300004, J11 691321300004, J12 691321300004, J3 CONN_06_SMD_FEMALE, J4 SDCARD_SLOT_TF-115K, J5 691321300004, J6 691321300004, J7 691321300004, J8 691321300004, J9 691321300004, Q1 FDD4141TO252, Q2 32.768kHz, U1 74HC165PW, U2 USBLC6-2SC6, U3 74HC595, U4 LD1117S33, U5 ATSAMD21G-A, X1 CONN_02, X2 25MHz, X3 RJ45_MAGNETICS_LED_HR871181A

Commit message: Updated hardware design files
Parts:
- added R22: 330R, OPL_Resistor:SMD-RES-330R-1%-1/10W(0603)
- added TP40, TP41, TP42: TESTPOINT_D1.6, PonoorExperiments:TESTPOINT_D1.6
- C105, C107, C109, C111, C65, C67, C69, C71: value 220nF -> 220nf; device Seeed-Capacitor:CERAMIC-10NF-50V-10%-X7R(0402) -> OPL_Capacitor:CERAMIC-220NF-25V-10%-X7R(0603)
- C23, C28: device Seeed-Capacitor:CERAMIC-10NF-50V-10%-X7R(0402) -> OPL_Capacitor:CERAMIC-10NF-50V-10%-X7R(0603)
- R3, R5, R9: value 10K 1/10W -> 100K 1/10W
- TP7: value TESTPOINT_3X1 -> TESTPOINT_D1.6; device PonoorExperiments:TESTPOINT_3X1 -> PonoorExperiments:TESTPOINT_D1.6
Connections:
- removed net D2: TP7.1, U5.PA14(XIN/SER2:2+)
- new net 74HC165_MOSI: U1.DS, U5.PA14(XIN/SER2:2+)
- new net N$46: 3.3V.+, R22.1
- net GND: no longer U1.DS
- net N$27: now also R22.2; no longer 3.3V.+
- net N$34: now also TP7.1
- net N$40: now also TP40.1
- net N$42: now also TP41.1
- net N$44: now also TP42.1
Other:
- moved on the sheet: 3.3V, C1, C7, ID, J2, J3, R3, R6, R7, RN1A, RN1B, RN1C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
