File: hardware/STEP800_brakeConverter/STEP800_brakeConverter.kicad_sch (KiCad schematic)
At the start: 11 parts, among them J1 Conn_02x05_Odd_Even, J2 Conn_02x03_Odd_Even, J3 Conn_02x03_Odd_Even, J4 Barrel_Jack_Switch, J5 Conn_01x02, J6 Conn_01x02, J7 Conn_01x02

Commit message: generate the board layout
Parts:
- H1, H2, H3, H4: footprint (none) -> MountingHole:MountingHole_3.2mm_M3_Pad_TopBottom
- J1: footprint (none) -> Connector_IDC:IDC-Header_2x05_P2.54mm_Vertical
- J2, J3: footprint (none) -> Connector_IDC:IDC-Header_2x03_P2.54mm_Vertical
- J4: footprint (none) -> Connector_BarrelJack:BarrelJack_GCT_DCJ200-10-A_Horizontal
- J5, J6, J7: footprint (none) -> Connector_Phoenix_MC:PhoenixContact_MCV_1,5_2-G-3.81_1x02_P3.81mm_Vertical
Changed lines of the file:
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@@
       (effects (font (size 1.27 1.27)) (justify left))
     )
-    (property "Footprint" "" (at 105.41 118.11 0)
+    (property "Footprint" "Connector_Phoenix_MC:PhoenixContact_MCV_1,5_2-G-3.81_1x02_P3.81mm_Vertical" (at 105.41 118.11 0)
       (effects (font (size 1.27 1.27)) hide)
     )
@@
       (effects (font (size 1.27 1.27)))
     )
-    (property "Footprint" "" (at 114.3 48.26 0)
+    (property "Footprint" "Connector_IDC:IDC-Header_2x03_P2.54mm_Vertical" (at 114.3 48.26 0)
       (effects (font (size 1.27 1.27)) hide)
     )
@@
       (effects (font (size 1.27 1.27)))
     )
-    (property "Footprint" "" (at 153.67 68.58 0)
+    (property "Footprint" "MountingHole:MountingHole_3.2mm_M3_Pad_TopBottom" (at 153.67 68.58 0)
       (effects (font (size 1.27 1.27)) hide)
     )
@@
       (effects (font (size 1.27 1.27)) (justify left))
     )
-    (property "Footprint" "" (at 105.41 102.87 0)
+    (property "Footprint" "Connector_Phoenix_MC:PhoenixContact_MCV_1,5_2-G-3.81_1x02_P3.81mm_Vertical" (at 105.41 102.87 0)
       (effects (font (size 1.27 1.27)) hide)
     )
@@
       (effects (font (size 1.27 1.27)))
     )
-    (property "Footprint" "" (at 153.67 50.8 0)
+    (property "Footprint" "MountingHole:MountingHole_3.2mm_M3_Pad_TopBottom" (at 153.67 50.8 0)
       (effects (font (size 1.27 1.27)) hide)
     )
@@
       (effects (font (size 1.27 1.27)))
     )
-    (property "Footprint" "" (at 153.67 59.69 0)
+    (property "Footprint" "MountingHole:MountingHole_3.2mm_M3_Pad_TopBottom" (at 153.67 59.69 0)
       (effects (font (size 1.27 1.27)) hide)
     )
@@
       (effects (font (size 1.27 1.27)))
     )
-    (property "Footprint" "" (at 71.12 105.156 0)
+    (property "Footprint" "Connector_BarrelJack:BarrelJack_GCT_DCJ200-10-A_Horizontal" (at 71.12 105.156 0)
       (effects (font (size 1.27 1.27)) hide)
     )
@@
       (effects (font (size 1.27 1.27)))
     )
-    (property "Footprint" "" (at 72.39 125.73 0)
+    (property "Footprint" "Connector_Phoenix_MC:PhoenixContact_MCV_1,5_2-G-3.81_1x02_P3.81mm_Vertical" (at 72.39 125.73 0)
       (effects (font (size 1.27 1.27)) hide)
     )
@@
       (effects (font (size 1.27 1.27)))
     )
-    (property "Footprint" "" (at 114.3 72.39 0)
+    (property "Footprint" "Connector_IDC:IDC-Header_2x03_P2.54mm_Vertical" (at 114.3 72.39 0)
       (effects (font (size 1.27 1.27)) hide)
     )
@@
       (effects (font (size 1.27 1.27)))
     )
-    (property "Footprint" "" (at 73.66 49.53 0)
+    (property "Footprint" "Connector_IDC:IDC-Header_2x05_P2.54mm_Vertical" (at 73.66 49.53 0)
       (effects (font (size 1.27 1.27)) hide)
     )
@@
       (effects (font (size 1.27 1.27)))
     )
-    (property "Footprint" "" (at 153.67 77.47 0)
-      (effects (font (size 1.27 1.27)) hide)
-    )
+    (property "Footprint" "MountingHole:MountingHole_3.2mm_M3_Pad_TopBottom" (at 153.67 77.47 0)
+      (effects (font (size 1.27 1.27)) hide)
+    )
